Commit message: add suction

File: cliport/environments/assets/ur5/suction/suction-base.urdf (robot description, URDF)
Before this commit: robot suction-base.urdf, 2 links, 1 joints
Links:
- link baseLink: mass .1 -> .05
- link midLink: mass .1 -> .05

File: cliport/environments/assets/ur5/suction/suction-head.urdf (robot description, URDF)
Before this commit: robot suction-head.urdf, 2 links, 1 joints
Links:
- link headLink: mass .1 -> .05
- link tipLink: mass .1 -> .05
