Commit message: add locobot update

File: cliport/environments/assets/locobot_description/locobot.urdf (robot description, URDF)
Before this commit: robot locobot, 26 links, 25 joints
Links:
- removed link finger_l
- removed link finger_r
Joints:
- removed joint joint_6
- removed joint joint_7

Commit message: add suction

File: cliport/environments/assets/locobot_description/locobot.urdf (robot description, URDF)
Before this commit: robot locobot, 24 links, 23 joints
Links:
- added link finger, mass .05; collision mesh filename=suction/head.obj scale=0.001 0.001 0.001; visual mesh filename=suction/head.obj scale=0.001 0.001 0.001
- added link tipLink, mass .05; collision cylinder length=0.028 radius=0.001; visual mesh filename=suction/tip.obj scale=0.001 0.001 0.001
Joints:
- added joint joint_6: type fixed, parent gripper_link, child finger, origin xyz=0.07285 0 0.0050143 rpy=1.57 0 1.57, axis 0 1 0, limit lower=-1 upper=0 effort=1 velocity=1
- added joint tipJoint: type fixed, parent finger, child tipLink, origin xyz=0.0 0.0 0.029 rpy=0.0 0.0 0.0, axis 0 0 1, limit lower=-6.28318530718 upper=6.28318530718 effort=150.0 velocity=3.15

Commit message: suction pick place

File: cliport/environments/assets/locobot_description/locobot.urdf (robot description, URDF)
Before this commit: robot locobot, 26 links, 25 joints
Links:
- removed link finger
- removed link tipLink
Joints:
- removed joint joint_6
- removed joint tipJoint
